Commit message: Implement caster rotation along all three axes

File: robocake_description/urdf/casters.urdf.xacro (robot description, xacro)
@@ -10,8 +10,20 @@
                                                          izz="0.129104"/>
     </link>
-    <joint name="${prefix}_caster_to_base" type="continuous">
+    <joint name="${prefix}_caster_x" type="continuous">
       <parent link="base"/>
       <origin xyz="${reflect * 0.049191} 0 -0.036909"/>
+      <axis xyz="1 0 0"/>
+      <child link="${prefix}_caster_x_to_y"/>
+    </joint>
+    <xacro:dummy_link name="${prefix}_caster_x_to_y"/>
+    <joint name="${prefix}_caster_y" type="continuous">
+      <parent link="${prefix}_caster_x_to_y"/>
       <axis xyz="0 1 0"/>
+      <child link="${prefix}_caster_y_to_z"/>
+    </joint>
+    <xacro:dummy_link name="${prefix}_caster_y_to_z"/>
+    <joint name="${prefix}_caster_z" type="continuous">
+      <parent link="${prefix}_caster_y_to_z"/>
+      <axis xyz="0 0 1"/>
       <child link="${prefix}_caster"/>
     </joint>

File: robocake_description/urdf/common.xacro (robot description, xacro)
@@ -47,3 +47,19 @@
     </inertial>
   </xacro:macro>
+  <!--
+      Creates a dummy link with no geometry, low mass and low inertia. Used for
+      emulating joints with multiple rotation axes. Gazebo requires mass and
+      inertial tensor to be non-zero, otherwise the link is not created in the
+      simulation at all or behaves incorrectly.
+  -->
+  <xacro:macro name="dummy_link" params="name">
+    <link name="${name}">
+      <inertial>
+        <mass value="0.001"/>
+        <inertia ixx="1e-12" ixy="0"     ixz="0"
+                             iyy="1e-12" iyz="0"
+                                         izz="1e-12"/>
+      </inertial>
+    </link>
+  </xacro:macro>
 </robot>
