Commit message: Add camera sensors

File: robocake_description/urdf/common.xacro (robot description, xacro)
@@ -60,9 +60,9 @@
       for small angles.
   -->
-  <xacro:macro name="gazebo_sensor"
+  <xacro:macro name="gazebo_proximity_sensor"
                params="name angle min_range max_range type">
     <gazebo reference="${name}_link">
       <sensor type="ray" name="${name}_sensor">
-        <visualize>true</visualize>
+        <visualize>false</visualize>
         <ray>
           <scan>

File: robocake_description/urdf/infrared.urdf.xacro (robot description, xacro)
@@ -31,6 +31,8 @@
         sensor's range.
     -->
-    <xacro:gazebo_sensor name="proximity_${side}" angle="${2 / 180 * pi}"
-                         min_range="0.005941" max_range="0.05" type="infrared"/>
+    <xacro:gazebo_proximity_sensor name="proximity_${side}"
+                                   angle="${2 / 180 * pi}"
+                                   min_range="0.005941" max_range="0.05"
+                                   type="infrared"/>
   </xacro:macro>
 </robot>

File: robocake_description/urdf/reflectance.urdf.xacro (robot description, xacro)
@@ -10,5 +10,5 @@
       <collision>
         <geometry>
-          <box size="0.0145 0.008 0.002"/>
+          <box size="0.002 0.008 0.0145"/>
         </geometry>
       </collision>
@@ -23,7 +23,25 @@
       <origin xyz="${0.085334 if reflect else 0.028881}
                    ${reflect * 0.027562}
-                   -0.031259"/>
+                   -0.031259"
+              rpy="0 ${pi / 2} 0"/>
       <child link="reflectance_${side}_link"/>
     </joint>
+    <gazebo reference="reflectance_${side}_link">
+      <sensor type="camera" name="${side}_camera">
+        <visualize>false</visualize>
+        <camera name="${side}_camera">
+          <clip>
+            <near>0.001</near>
+          </clip>
+          <image>
+            <width>1</width>
+            <height>1</height>
+          </image>
+        </camera>
+        <plugin name="gazebo_ros_camera" filename="libgazebo_ros_camera.so">
+          <cameraName>${side}_camera</cameraName>
+        </plugin>
+      </sensor>
+    </gazebo>
   </xacro:macro>
 </robot>

File: robocake_description/urdf/ultrasonic.urdf.xacro (robot description, xacro)
@@ -20,6 +20,8 @@
       <child link="proximity_front_link"/>
     </joint>
-    <xacro:gazebo_sensor name="proximity_front" angle="${5 / 180 * pi}"
-                       min_range="0.02" max_range="4" type="ultrasound"/>
+    <xacro:gazebo_proximity_sensor name="proximity_front"
+                                   angle="${5 / 180 * pi}"
+                                   min_range="0.02" max_range="0.8"
+                                   type="ultrasound"/>
   </xacro:macro>
 </robot>
