Commit message: Use primitives for collisions where possible

File: robocake_description/urdf/base.urdf.xacro (robot description, xacro)
@@ -2,5 +2,6 @@
 <robot xmlns:xacro="http://www.ros.org/wiki/xacro" name="robocake">
   <link name="base">
-    <xacro:mesh_geometry name="base"/>
+    <xacro:mesh_visual name="base"/>
+    <xacro:mesh_collision name="base"/>
     <xacro:mesh_inertia mass="0.5" scaling="10" volume="0.213995"
                         x="0.006792" y="0.000060" z="0.016779"

File: robocake_description/urdf/casters.urdf.xacro (robot description, xacro)
@@ -3,5 +3,10 @@
   <xacro:macro name="caster" params="prefix reflect">
     <link name="${prefix}_caster">
-      <xacro:mesh_geometry name="caster" use_collision_mesh="false"/>
+      <xacro:mesh_visual name="caster"/>
+      <collision>
+        <geometry>
+          <sphere radius="0.005995"/>
+        </geometry>
+      </collision>
       <xacro:mesh_inertia mass="0.01" scaling="100" volume="0.899919"
                           x="0.000007" y="0.000028" z="-0.000015"

File: robocake_description/urdf/common.xacro (robot description, xacro)
@@ -1,26 +1,17 @@
 <?xml version="1.0"?>
 <robot xmlns:xacro="http://www.ros.org/wiki/xacro">
-  <xacro:macro name="mesh_geometry" params="name use_collision_mesh:=true">
-    <xacro:property name="visual_mesh" value="visual/${name}.dae"/>
-    <!--
-        If use_collision_mesh is true (defaut), use a separate simplified mesh
-        for collision detection from /collision/ subdirectory. Otherwise, use
-        the same mesh as the one displayed visually.
-    -->
-    <xacro:if value="${use_collision_mesh}">
-      <xacro:property name="collision_mesh" value="collision/${name}.dae"/>
-    </xacro:if>
-    <xacro:unless value="${use_collision_mesh}">
-      <xacro:property name="collision_mesh" value="${visual_mesh}"/>
-    </xacro:unless>
+  <xacro:macro name="mesh_visual" params="name">
     <visual>
       <geometry>
-        <mesh filename="package://robocake_description/meshes/${visual_mesh}"/>
+        <mesh
+          filename="package://robocake_description/meshes/visual/${name}.dae"/>
       </geometry>
     </visual>
+  </xacro:macro>
+  <xacro:macro name="mesh_collision" params="name">
     <collision>
       <geometry>
         <mesh
-          filename="package://robocake_description/meshes/${collision_mesh}"/>
+          filename="package://robocake_description/meshes/collision/${name}.dae"/>
       </geometry>
     </collision>

File: robocake_description/urdf/infrared.urdf.xacro (robot description, xacro)
@@ -7,5 +7,11 @@
   <xacro:macro name="infrared" params="side reflect">
     <link name="proximity_${side}">
-      <xacro:mesh_geometry name="infrared"/>
+      <xacro:mesh_visual name="infrared"/>
+      <collision>
+        <origin xyz="0.001551 -0.000007 -0.001367"/>
+        <geometry>
+          <box size="0.007902 0.00630 0.013642"/>
+        </geometry>
+      </collision>
       <xacro:mesh_inertia mass="0.01" scaling="100" volume="0.943720"
                         x="0.006637" y="-0.000480" z="-0.183167"
@@ -16,5 +22,5 @@
     <joint name="proximity_${side}_to_base" type="fixed">
       <parent link="base"/>
-      <origin xyz="0.035447 ${reflect * -0.06118} 0.005715"
+      <origin xyz="0.034096 ${reflect * -0.058848} 0.005497"
               rpy="0 0 ${reflect * 5 / 3 * pi}"/>
       <child link="proximity_${side}"/>

File: robocake_description/urdf/ultrasonic.urdf.xacro (robot description, xacro)
@@ -6,5 +6,6 @@
   -->
   <link name="proximity_front">
-    <xacro:mesh_geometry name="ultrasonic"/>
+    <xacro:mesh_visual name="ultrasonic"/>
+    <xacro:mesh_collision name="ultrasonic"/>
     <xacro:mesh_inertia mass="0.02" scaling="10" volume="0.005512"
                         x="0.002263" y="-0.000840" z="0.013641"

File: robocake_description/urdf/wheels.urdf.xacro (robot description, xacro)
@@ -3,5 +3,11 @@
   <xacro:macro name="wheel" params="prefix reflect">
     <link name="${prefix}_wheel">
-      <xacro:mesh_geometry name="wheel"/>
+      <xacro:mesh_visual name="wheel"/>
+      <collision>
+        <origin xyz="0.000998 0.000001 -0.000002" rpy="0 ${pi / 2} 0"/>
+        <geometry>
+          <cylinder radius="0.022131" length="0.017986"/>
+        </geometry>
+      </collision>
       <xacro:mesh_inertia mass="0.03" scaling="10" volume="0.015398"
                           x="0.010317" y="-0.000083" z="-0.000017"

Commit message: Separate robots into different files

File: robocake_description/urdf/base.urdf.xacro (robot description, xacro)
@@ -1,8 +1,8 @@
 <?xml version="1.0"?>
 <robot xmlns:xacro="http://www.ros.org/wiki/xacro" name="robocake">
-  <xacro:macro name="base">
+  <xacro:macro name="base" params="name">
     <link name="base_link">
-      <xacro:mesh_visual name="base"/>
-      <xacro:mesh_collision name="base"/>
+      <xacro:mesh_visual name="base_${name}"/>
+      <xacro:mesh_collision name="base_${name}"/>
       <xacro:mesh_inertia mass="0.5" scaling="10" volume="0.213995"
                           x="0.006792" y="0.000060" z="0.016779"
