Commit message: Implement collision and inertia for base link

File: robocake_description/robots/robocake.urdf.xacro (robot description, xacro)
@@ -1,4 +1,5 @@
 <?xml version="1.0"?>
 <robot xmlns:xacro="http://www.ros.org/wiki/xacro" name="robocake">
+  <xacro:include filename="$(find robocake_description)/urdf/common.xacro"/>
   <link name="base">
     <visual>
@@ -9,11 +10,13 @@
     <collision>
       <geometry>
-        <mesh filename="package://robocake_description/meshes/main/base.dae"/>
+        <mesh
+          filename="package://robocake_description/meshes/collision/base.stl"/>
       </geometry>
     </collision>
-    <inertial>
-      <mass value="1"/>
-      <inertia ixx="0.1" ixy="0" ixz="0" iyy="0.1" iyz="0" izz="0.1"/>
-    </inertial>
+    <xacro:mesh_inertia mass="1" scaling="10" volume="0.214749"
+                        x="0.006736"   y="-0.000233"   z="-0.023669"
+                        ixx="0.057916" ixy="-0.000012" ixz="0.000804"
+                                       iyy="0.059992"  iyz="-0.000007"
+                                                       izz="0.085993"/>
   </link>
 </robot>

Commit message: Implement wheels

File: robocake_description/robots/robocake.urdf.xacro (robot description, xacro)
@@ -2,21 +2,5 @@
 <robot xmlns:xacro="http://www.ros.org/wiki/xacro" name="robocake">
   <xacro:include filename="$(find robocake_description)/urdf/common.xacro"/>
-  <link name="base">
-    <visual>
-      <geometry>
-        <mesh filename="package://robocake_description/meshes/main/base.dae"/>
-      </geometry>
-    </visual>
-    <collision>
-      <geometry>
-        <mesh
-          filename="package://robocake_description/meshes/collision/base.stl"/>
-      </geometry>
-    </collision>
-    <xacro:mesh_inertia mass="1" scaling="10" volume="0.214749"
-                        x="0.006736"   y="-0.000233"   z="-0.023669"
-                        ixx="0.057916" ixy="-0.000012" ixz="0.000804"
-                                       iyy="0.059992"  iyz="-0.000007"
-                                                       izz="0.085993"/>
-  </link>
+  <xacro:include filename="$(find robocake_description)/urdf/base.urdf.xacro"/>
+  <xacro:include filename="$(find robocake_description)/urdf/wheel.urdf.xacro"/>
 </robot>

File: robocake_description/urdf/common.xacro (robot description, xacro)
@@ -1,9 +1,23 @@
 <?xml version="1.0"?>
 <robot xmlns:xacro="http://www.ros.org/wiki/xacro">
+  <xacro:macro name="mesh_geometry" params="name">
+    <visual>
+      <geometry>
+        <mesh
+          filename="package://robocake_description/meshes/visual/${name}.dae"/>
+      </geometry>
+    </visual>
+    <collision>
+      <geometry>
+        <mesh
+          filename="package://robocake_description/meshes/collision/${name}.stl"/>
+      </geometry>
+    </collision>
+  </xacro:macro>
   <!--
-    Generates inertial tag for a mesh link based on meshlab output.
-      scaling - temporary scaling applied in meshlab to increase precision.
-      x, y, z - center of mass.
-      ixx..izz - above-diagonal elements of the inertia tensor.
+      Generates inertial tag for a mesh link based on meshlab output.
+        scaling - temporary scaling applied in meshlab to increase precision.
+        x, y, z - center of mass.
+        ixx..izz - above-diagonal elements of the inertia tensor.
   -->
   <xacro:macro name="mesh_inertia"

Commit message: Adjust wheel clearance and positioning

File: robocake_description/robots/robocake.urdf.xacro (robot description, xacro)
@@ -3,4 +3,5 @@
   <xacro:include filename="$(find robocake_description)/urdf/common.xacro"/>
   <xacro:include filename="$(find robocake_description)/urdf/base.urdf.xacro"/>
-  <xacro:include filename="$(find robocake_description)/urdf/wheel.urdf.xacro"/>
+  <xacro:include
+    filename="$(find robocake_description)/urdf/wheels.urdf.xacro"/>
 </robot>

File: robocake_description/urdf/base.urdf.xacro (robot description, xacro)
@@ -3,9 +3,9 @@
   <link name="base">
     <xacro:mesh_geometry name="base"/>
-    <xacro:mesh_inertia mass="1" scaling="10" volume="0.216312"
-                        x="0.006792" y="-0.000125" z="0.013660"
-                        ixx="0.058219" ixy="-0.000005" ixz="0.000802"
-                                       iyy="0.061790"  iyz="-0.000001"
-                                                       izz="0.087097"/>
+    <xacro:mesh_inertia mass="1" scaling="10" volume="0.213995"
+                        x="0.006792" y="0.000060" z="0.016779"
+                        ixx="0.057859" ixy="0.000003" ixz="0.000809"
+                                       iyy="0.061351"  iyz="0.000007"
+                                                       izz="0.086716"/>
   </link>
 </robot>

File: robocake_description/urdf/wheels.urdf.xacro (robot description, xacro)
@@ -5,5 +5,5 @@
       <xacro:mesh_geometry name="wheel"/>
       <xacro:mesh_inertia mass="1" scaling="10" volume="0.015398"
-                          x="0.010317" y="-0.000085" z="-0.000002"
+                          x="0.010317" y="-0.000083" z="-0.000017"
                           ixx="0.000466" ixy="0"         ixz="0"
                                          iyy="0.000272"  iyz="0"
@@ -12,5 +12,6 @@
     <joint name="${prefix}_wheel_to_base" type="continuous">
       <parent link="base"/>
-      <origin xyz="-0.001 ${reflect * 0.043} -0.025" rpy="0 0 ${reflect * pi / 2}"/>
+      <origin xyz="0.00002 ${reflect * 0.042459} -0.020922"
+              rpy="0 0 ${reflect * pi / 2}"/>
       <child link="${prefix}_wheel"/>
     </joint>

Commit message: Implement casters

File: robocake_description/robots/robocake.urdf.xacro (robot description, xacro)
@@ -5,3 +5,5 @@
   <xacro:include
     filename="$(find robocake_description)/urdf/wheels.urdf.xacro"/>
+  <xacro:include
+    filename="$(find robocake_description)/urdf/casters.urdf.xacro"/>
 </robot>

File: robocake_description/urdf/common.xacro (robot description, xacro)
@@ -1,9 +1,20 @@
 <?xml version="1.0"?>
 <robot xmlns:xacro="http://www.ros.org/wiki/xacro">
-  <xacro:macro name="mesh_geometry" params="name">
+  <xacro:macro name="mesh_geometry" params="name use_collision_mesh:=true">
+    <xacro:property name="visual_mesh" value="visual/${name}.dae"/>
+    <!--
+        If use_collision_mesh is true (defaut), use a separate simplified mesh
+        for collision detection from /collision/ subdirectory. Otherwise, use
+        the same mesh as the one displayed visually.
+    -->
+    <xacro:if value="${use_collision_mesh}">
+      <xacro:property name="collision_mesh" value="collision/${name}.dae"/>
+    </xacro:if>
+    <xacro:unless value="${use_collision_mesh}">
+      <xacro:property name="collision_mesh" value="${visual_mesh}"/>
+    </xacro:unless>
     <visual>
       <geometry>
-        <mesh
-          filename="package://robocake_description/meshes/visual/${name}.dae"/>
+        <mesh filename="package://robocake_description/meshes/${visual_mesh}"/>
       </geometry>
     </visual>
@@ -11,5 +22,5 @@
       <geometry>
         <mesh
-          filename="package://robocake_description/meshes/collision/${name}.dae"/>
+          filename="package://robocake_description/meshes/${collision_mesh}"/>
       </geometry>
     </collision>

Commit message: Add differential drive controller

File: robocake_description/robots/robocake.urdf.xacro (robot description, xacro)
@@ -7,3 +7,8 @@
   <xacro:include
     filename="$(find robocake_description)/urdf/casters.urdf.xacro"/>
+  <gazebo>
+    <plugin name="gazebo_ros_control" filename="libgazebo_ros_control.so">
+      <legacyModeNS>true</legacyModeNS>
+    </plugin>
+  </gazebo>
 </robot>

File: robocake_description/urdf/wheels.urdf.xacro (robot description, xacro)
@@ -14,6 +14,14 @@
       <origin xyz="0.00002 ${reflect * 0.042459} -0.020922"
               rpy="0 0 ${reflect * pi / 2}"/>
+      <axis xyz="${reflect} 0 0"/>
       <child link="${prefix}_wheel"/>
     </joint>
+    <transmission name="${prefix}_wheel_transmission">
+      <type>transmission_interface/SimpleTransmission</type>
+      <actuator name="${prefix}_wheel_actuator"/>
+      <joint name="${prefix}_wheel_to_base">
+        <hardwareInterface>hardware_interface/VelocityJointInterface</hardwareInterface>
+      </joint>
+    </transmission>
   </xacro:macro>
   <xacro:wheel prefix="left" reflect="1"/>

Commit message: Move sensor definition to a macro

File: robocake_description/robots/robocake.urdf.xacro (robot description, xacro)
@@ -8,5 +8,5 @@
     filename="$(find robocake_description)/urdf/casters.urdf.xacro"/>
   <xacro:include
-    filename="$(find robocake_description)/urdf/hcsr04.urdf.xacro"/>
+    filename="$(find robocake_description)/urdf/ultrasonic.urdf.xacro"/>
   <gazebo>
     <plugin name="gazebo_ros_control" filename="libgazebo_ros_control.so">

File: robocake_description/urdf/common.xacro (robot description, xacro)
@@ -63,3 +63,35 @@
     </link>
   </xacro:macro>
+  <xacro:macro name="gazebo_sensor"
+               params="name angle:=0 min_range max_range samples:=1 type">
+    <gazebo reference="${name}">
+      <sensor type="ray" name="${name}_sensor">
+        <visualize>true</visualize>
+        <ray>
+          <scan>
+            <horizontal>
+              <samples>${samples}</samples>
+              <min_angle>${-angle / 2}</min_angle>
+              <max_angle>${angle / 2}</max_angle>
+            </horizontal>
+            <vertical>
+              <samples>${samples}</samples>
+              <min_angle>${-angle / 2}</min_angle>
+              <max_angle>${angle / 2}</max_angle>
+            </vertical>
+          </scan>
+          <range>
+            <min>${min_range}</min>
+            <max>${max_range}</max>
+          </range>
+        </ray>
+        <plugin filename="libgazebo_ros_range.so" name="gazebo_ros_range">
+          <topicName>${name}</topicName>
+          <frameName>${name}</frameName>
+          <fov>${angle}</fov>
+          <radiation>${type}</radiation>
+        </plugin>
+      </sensor>
+    </gazebo>
+  </xacro:macro>
 </robot>

Commit message: Move macro calls to make them more reusable

File: robocake_description/robots/robocake.urdf.xacro (robot description, xacro)
@@ -3,12 +3,19 @@
   <xacro:include filename="$(find robocake_description)/urdf/common.xacro"/>
   <xacro:include filename="$(find robocake_description)/urdf/base.urdf.xacro"/>
+  <xacro:include filename="$(find robocake_description)/urdf/wheel.urdf.xacro"/>
   <xacro:include
-    filename="$(find robocake_description)/urdf/wheels.urdf.xacro"/>
-  <xacro:include
-    filename="$(find robocake_description)/urdf/casters.urdf.xacro"/>
+    filename="$(find robocake_description)/urdf/caster.urdf.xacro"/>
   <xacro:include
     filename="$(find robocake_description)/urdf/ultrasonic.urdf.xacro"/>
   <xacro:include
     filename="$(find robocake_description)/urdf/infrared.urdf.xacro"/>
+  <xacro:base/>
+  <xacro:wheel prefix="left" reflect="1"/>
+  <xacro:wheel prefix="right" reflect="-1"/>
+  <xacro:caster prefix="front" reflect="1"/>
+  <xacro:caster prefix="back" reflect="-1"/>
+  <xacro:ultrasonic/>
+  <xacro:infrared side="left" reflect="1"/>
+  <xacro:infrared side="right" reflect="-1"/>
   <gazebo>
     <plugin name="gazebo_ros_control" filename="libgazebo_ros_control.so">

File: robocake_description/urdf/base.urdf.xacro (robot description, xacro)
@@ -1,12 +1,14 @@
 <?xml version="1.0"?>
 <robot xmlns:xacro="http://www.ros.org/wiki/xacro" name="robocake">
-  <link name="base">
-    <xacro:mesh_visual name="base"/>
-    <xacro:mesh_collision name="base"/>
-    <xacro:mesh_inertia mass="0.5" scaling="10" volume="0.213995"
-                        x="0.006792" y="0.000060" z="0.016779"
-                        ixx="0.057859" ixy="0.000003" ixz="0.000809"
-                                       iyy="0.061351"  iyz="0.000007"
-                                                       izz="0.086716"/>
-  </link>
+  <xacro:macro name="base">
+    <link name="base_link">
+      <xacro:mesh_visual name="base"/>
+      <xacro:mesh_collision name="base"/>
+      <xacro:mesh_inertia mass="0.5" scaling="10" volume="0.213995"
+                          x="0.006792" y="0.000060" z="0.016779"
+                          ixx="0.057859" ixy="0.000003" ixz="0.000809"
+                                         iyy="0.061351" iyz="0.000007"
+                                                        izz="0.086716"/>
+    </link>
+  </xacro:macro>
 </robot>

File: robocake_description/urdf/caster.urdf.xacro (robot description, xacro)
@@ -2,5 +2,5 @@
 <robot xmlns:xacro="http://www.ros.org/wiki/xacro">
   <xacro:macro name="caster" params="prefix reflect">
-    <link name="${prefix}_caster">
+    <link name="${prefix}_caster_link">
       <xacro:mesh_visual name="caster"/>
       <collision>
@@ -15,24 +15,27 @@
                                                          izz="0.129104"/>
     </link>
-    <joint name="${prefix}_caster_x" type="continuous">
-      <parent link="base"/>
+    <!--
+        Since the ball caster has three degrees of freedom while continuous
+        joint only has one, it is implemented as three separate joints connected
+        with dummy links.
+    -->
+    <xacro:dummy_link name="${prefix}_caster_x_to_y_link"/>
+    <joint name="${prefix}_caster_x_joint" type="continuous">
+      <parent link="base_link"/>
       <origin xyz="${reflect * 0.049191} 0 -0.036909"/>
       <axis xyz="1 0 0"/>
-      <child link="${prefix}_caster_x_to_y"/>
+      <child link="${prefix}_caster_x_to_y_link"/>
     </joint>
-    <xacro:dummy_link name="${prefix}_caster_x_to_y"/>
-    <joint name="${prefix}_caster_y" type="continuous">
-      <parent link="${prefix}_caster_x_to_y"/>
+    <xacro:dummy_link name="${prefix}_caster_y_to_z_link"/>
+    <joint name="${prefix}_caster_y_joint" type="continuous">
+      <parent link="${prefix}_caster_x_to_y_link"/>
       <axis xyz="0 1 0"/>
-      <child link="${prefix}_caster_y_to_z"/>
+      <child link="${prefix}_caster_y_to_z_link"/>
     </joint>
-    <xacro:dummy_link name="${prefix}_caster_y_to_z"/>
-    <joint name="${prefix}_caster_z" type="continuous">
-      <parent link="${prefix}_caster_y_to_z"/>
+    <joint name="${prefix}_caster_z_joint" type="continuous">
+      <parent link="${prefix}_caster_y_to_z_link"/>
       <axis xyz="0 0 1"/>
-      <child link="${prefix}_caster"/>
+      <child link="${prefix}_caster_link"/>
     </joint>
   </xacro:macro>
-  <xacro:caster prefix="front" reflect="1"/>
-  <xacro:caster prefix="back" reflect="-1"/>
 </robot>

File: robocake_description/urdf/common.xacro (robot description, xacro)
@@ -62,5 +62,5 @@
   <xacro:macro name="gazebo_sensor"
                params="name angle min_range max_range type">
-    <gazebo reference="${name}">
+    <gazebo reference="${name}_link">
       <sensor type="ray" name="${name}_sensor">
         <visualize>true</visualize>
@@ -85,5 +85,5 @@
         <plugin filename="libgazebo_ros_range.so" name="gazebo_ros_range">
           <topicName>${name}</topicName>
-          <frameName>${name}</frameName>
+          <frameName>${name}_link</frameName>
           <fov>${angle}</fov>
           <radiation>${type}</radiation>

File: robocake_description/urdf/infrared.urdf.xacro (robot description, xacro)
@@ -6,5 +6,5 @@
   -->
   <xacro:macro name="infrared" params="side reflect">
-    <link name="proximity_${side}">
+    <link name="proximity_${side}_link">
       <xacro:mesh_visual name="infrared"/>
       <collision>
@@ -20,9 +20,9 @@
                                                        izz="0.120043"/>
     </link>
-    <joint name="proximity_${side}_to_base" type="fixed">
-      <parent link="base"/>
+    <joint name="proximity_${side}_joint" type="fixed">
+      <parent link="base_link"/>
       <origin xyz="0.034096 ${reflect * -0.058848} 0.005497"
               rpy="0 0 ${reflect * 5 / 3 * pi}"/>
-      <child link="proximity_${side}"/>
+      <child link="proximity_${side}_link"/>
     </joint>
     <!--
@@ -34,5 +34,3 @@
                          min_range="0.005941" max_range="0.05" type="infrared"/>
   </xacro:macro>
-  <xacro:infrared side="left" reflect="1"/>
-  <xacro:infrared side="right" reflect="-1"/>
 </robot>

File: robocake_description/urdf/ultrasonic.urdf.xacro (robot description, xacro)
@@ -5,19 +5,21 @@
       See https://cdn.sparkfun.com/datasheets/Sensors/Proximity/HCSR04.pdf
   -->
-  <link name="proximity_front">
-    <xacro:mesh_visual name="ultrasonic"/>
-    <xacro:mesh_collision name="ultrasonic"/>
-    <xacro:mesh_inertia mass="0.02" scaling="10" volume="0.005512"
-                        x="0.002263" y="-0.000840" z="0.013641"
-                        ixx="0.000112" ixy="0"        ixz="0"
-                                       iyy="0.000017" iyz="0"
-                                                      izz="0.000111"/>
-  </link>
-  <joint name="proximity_front_to_base" type="fixed">
-    <parent link="base"/>
-    <origin xyz="0.072431 0.000139 0.001164"/>
-    <child link="proximity_front"/>
-  </joint>
-  <xacro:gazebo_sensor name="proximity_front" angle="${5 / 180 * pi}"
+  <xacro:macro name="ultrasonic">
+    <link name="proximity_front_link">
+      <xacro:mesh_visual name="ultrasonic"/>
+      <xacro:mesh_collision name="ultrasonic"/>
+      <xacro:mesh_inertia mass="0.02" scaling="10" volume="0.005512"
+                          x="0.002263" y="-0.000840" z="0.013641"
+                          ixx="0.000112" ixy="0"        ixz="0"
+                                         iyy="0.000017" iyz="0"
+                                                        izz="0.000111"/>
+    </link>
+    <joint name="proximity_front_joint" type="fixed">
+      <parent link="base_link"/>
+      <origin xyz="0.072431 0.000139 0.001164"/>
+      <child link="proximity_front_link"/>
+    </joint>
+    <xacro:gazebo_sensor name="proximity_front" angle="${5 / 180 * pi}"
                        min_range="0.02" max_range="4" type="ultrasound"/>
+  </xacro:macro>
 </robot>

File: robocake_description/urdf/wheel.urdf.xacro (robot description, xacro)
@@ -2,5 +2,5 @@
 <robot xmlns:xacro="http://www.ros.org/wiki/xacro">
   <xacro:macro name="wheel" params="prefix reflect">
-    <link name="${prefix}_wheel">
+    <link name="${prefix}_wheel_link">
       <xacro:mesh_visual name="wheel"/>
       <collision>
@@ -16,20 +16,18 @@
                                                          izz="0.000272"/>
     </link>
-    <joint name="${prefix}_wheel_to_base" type="continuous">
-      <parent link="base"/>
+    <joint name="${prefix}_wheel_joint" type="continuous">
+      <parent link="base_link"/>
       <origin xyz="0.00002 ${reflect * 0.042459} -0.020922"
               rpy="0 0 ${reflect * pi / 2}"/>
       <axis xyz="${reflect} 0 0"/>
-      <child link="${prefix}_wheel"/>
+      <child link="${prefix}_wheel_link"/>
     </joint>
     <transmission name="${prefix}_wheel_transmission">
       <type>transmission_interface/SimpleTransmission</type>
       <actuator name="${prefix}_wheel_actuator"/>
-      <joint name="${prefix}_wheel_to_base">
+      <joint name="${prefix}_wheel_joint">
         <hardwareInterface>hardware_interface/VelocityJointInterface</hardwareInterface>
       </joint>
     </transmission>
   </xacro:macro>
-  <xacro:wheel prefix="left" reflect="1"/>
-  <xacro:wheel prefix="right" reflect="-1"/>
 </robot>
